Commit message: moveit is running now

File: euroc_manipulation_moveit/config/arm.urdf (robot description, URDF)
Before this commit: robot kuka_lwr, 12 links, 11 joints
Joints:
- removed joint joint1
- removed joint joint2
- removed joint joint3
- removed joint joint4
- removed joint joint5
- removed joint joint6
- removed joint joint7
- added joint lwr_joint_1: type revolute, parent base, child link1, origin xyz=0 0 0.31 rpy=0 0 0, axis 0 0 1, limit lower=-2.96705972839 upper=2.96705972839 effort=150 velocity=1.6
- added joint lwr_joint_2: type revolute, parent link1, child link2, origin xyz=0 0 0 rpy=1.57079632679 0 0, axis 0 0 1, limit lower=-2.09439510239 upper=2.09439510239 effort=150 velocity=1.6
- added joint lwr_joint_3: type revolute, parent link2, child link3, origin xyz=0 0.2 0 rpy=-1.57079632679 0 0, axis 0 0 1, limit lower=-2.96705972839 upper=2.96705972839 effort=150 velocity=1.6
- added joint lwr_joint_4: type revolute, parent link3, child link4, origin xyz=0 0 0.2 rpy=-1.57079632679 0 0, axis 0 0 1, limit lower=-2.09439510239 upper=2.09439510239 effort=150 velocity=1.6
- added joint lwr_joint_5: type revolute, parent link4, child link5, origin xyz=0 -0.2 0 rpy=1.57079632679 0 0, axis 0 0 1, limit lower=-2.96705972839 upper=2.96705972839 effort=150 velocity=1.6
- added joint lwr_joint_6: type revolute, parent link5, child link6, origin xyz=0 0 0.19 rpy=1.57079632679 0 0, axis 0 0 1, limit lower=-2.26892802759 upper=2.26892802759 effort=150 velocity=1.6
- added joint lwr_joint_7: type revolute, parent link6, child link7, origin xyz=0 0 0 rpy=-1.57079632679 0 0, axis 0 0 1, limit lower=-2.96705972839 upper=2.96705972839 effort=150 velocity=1.6
