Commit message: added cam frames

File: suturo_manipulation_moveit/config/arm.urdf (robot description, URDF)
Before this commit: robot kuka_lwr, 12 links, 11 joints
Links:
- removed link gripper
- added link gp, mass 1.2; collision box size=0.112000 0.083000 0.093000; visual mesh filename=package://euroc_c2_description/pg70_gripper/pg70_body.dae
Joints:
- joint gripper_joint: child gripper -> gp
- joint joint_before_finger1: parent gripper -> gp
- joint joint_before_finger2: parent gripper -> gp

Commit message: moved cam frames to arm urdf

File: suturo_manipulation_moveit/config/arm.urdf (robot description, URDF)
Before this commit: robot kuka_lwr, 12 links, 11 joints
Links:
- added link tdepth
- added link trgb
Joints:
- added joint tdepth_joint: type fixed, parent trgb, child tdepth, origin xyz=0 -0.04 0 rpy=0 0 0
- added joint trgb_joint: type fixed, parent gp, child trgb, origin xyz=-0.02 0.0565 -0.063 rpy=-1.5708 1.5708 0

Commit message: fixed some bugs

File: suturo_manipulation_moveit/config/arm.urdf (robot description, URDF)
Before this commit: robot kuka_lwr, 14 links, 13 joints
Links:
- removed link base
- added link lwr_base, mass 2.7; collision cylinder length=0.11 radius=0.07; visual mesh filename=package://euroc_c2_description/kuka_lwr/kuka-lwr-base.dae
Joints:
- joint base_joint: child base -> lwr_base
- joint lwr_joint_1: limit lower=-2.96705972839 upper=2.96705972839 effort=150 velocity=1.6 -> lower=-2.962 upper=2.962 effort=150 velocity=1.6; parent base -> lwr_base
- joint lwr_joint_2: limit lower=-2.09439510239 upper=2.09439510239 effort=150 velocity=1.6 -> lower=-2.09 upper=2.09 effort=150 velocity=1.6
- joint lwr_joint_3: limit lower=-2.96705972839 upper=2.96705972839 effort=150 velocity=1.6 -> lower=-2.962 upper=2.962 effort=150 velocity=1.6
- joint lwr_joint_4: limit lower=-2.09439510239 upper=2.09439510239 effort=150 velocity=1.6 -> lower=-2.09 upper=2.09 effort=150 velocity=1.6
- joint lwr_joint_5: limit lower=-2.96705972839 upper=2.96705972839 effort=150 velocity=1.6 -> lower=-2.962 upper=2.962 effort=150 velocity=1.6
- joint lwr_joint_6: limit lower=-2.26892802759 upper=2.26892802759 effort=150 velocity=1.6 -> lower=-1.7 upper=1.7 effort=150 velocity=1.6
- joint lwr_joint_7: limit lower=-2.96705972839 upper=2.96705972839 effort=150 velocity=1.6 -> lower=-2.962 upper=2.962 effort=150 velocity=1.6

Commit message: added moveable base in urdf

File: suturo_manipulation_moveit/config/arm.urdf (robot description, URDF)
Before this commit: robot kuka_lwr, 14 links, 13 joints
Links:
- added link lwr_base_x, mass 2.7
- added link lwr_base_y, mass 2.7
Joints:
- added joint base_axis_x: type prismatic, parent base_link, child lwr_base_x, origin xyz=0 0 0.015 rpy=0 0 0, axis 1.0 0 0, limit lower=-1 upper=1 effort=150 velocity=1.6
- added joint base_axis_y: type prismatic, parent lwr_base_x, child lwr_base_y, origin xyz=0 0 0.035 rpy=0 0 0, axis 0 1.0 0, limit lower=-1 upper=1 effort=150 velocity=1.6
- joint base_joint: parent base_link -> lwr_base_y

Commit message: axis instead of base_axis

File: suturo_manipulation_moveit/config/arm.urdf (robot description, URDF)
Before this commit: robot kuka_lwr, 16 links, 15 joints
Joints:
- removed joint base_axis_x
- removed joint base_axis_y
- added joint axis_x: type prismatic, parent base_link, child lwr_base_x, origin xyz=0 0 0.015 rpy=0 0 0, axis 1.0 0 0, limit lower=-0.92 upper=0.92 effort=150 velocity=1.6
- added joint axis_y: type prismatic, parent lwr_base_x, child lwr_base_y, origin xyz=0 0 0.035 rpy=0 0 0, axis 0 1.0 0, limit lower=-0.92 upper=0.92 effort=150 velocity=1.6

Commit message: muhmuh

File: suturo_manipulation_moveit/config/arm.urdf (robot description, URDF)
Before this commit: robot kuka_lwr, 16 links, 15 joints
Joints:
- joint axis_x: origin xyz=0 0 0.015 rpy=0 0 0 -> xyz=0 0 0.005 rpy=0 0 0
- joint axis_y: origin xyz=0 0 0.035 rpy=0 0 0 -> xyz=0 0 0 rpy=0 0 0

Commit message: cooler scheiß

File: suturo_manipulation_moveit/config/arm.urdf (robot description, URDF)
Before this commit: robot kuka_lwr, 16 links, 15 joints
Joints:
- joint lwr_joint_1: limit lower=-2.962 upper=2.962 effort=150 velocity=1.6 -> lower=-2.96 upper=2.96 effort=150 velocity=1.6
- joint lwr_joint_2: limit lower=-2.09 upper=2.09 effort=150 velocity=1.6 -> lower=-2.092 upper=2.092 effort=150 velocity=1.6
- joint lwr_joint_3: limit lower=-2.962 upper=2.962 effort=150 velocity=1.6 -> lower=-2.96 upper=2.96 effort=150 velocity=1.6
- joint lwr_joint_4: limit lower=-2.09 upper=2.09 effort=150 velocity=1.6 -> lower=-2.092 upper=2.092 effort=150 velocity=1.6
- joint lwr_joint_5: limit lower=-2.962 upper=2.962 effort=150 velocity=1.6 -> lower=-2.96 upper=2.96 effort=150 velocity=1.6
- joint lwr_joint_7: limit lower=-2.962 upper=2.962 effort=150 velocity=1.6 -> lower=-2.96 upper=2.96 effort=150 velocity=1.6

Commit message: added more output, decreased base joint max values

File: suturo_manipulation_moveit/config/arm.urdf (robot description, URDF)
Before this commit: robot kuka_lwr, 16 links, 15 joints
Joints:
- joint axis_x: limit lower=-0.92 upper=0.92 effort=150 velocity=1.6 -> lower=-0.9 upper=0.9 effort=150 velocity=1.6
- joint axis_y: limit lower=-0.92 upper=0.92 effort=150 velocity=1.6 -> lower=-0.9 upper=0.9 effort=150 velocity=1.6

Commit message: added more output

File: suturo_manipulation_moveit/config/arm.urdf (robot description, URDF)
Before this commit: robot kuka_lwr, 16 links, 15 joints
Joints:
- joint axis_x: limit lower=-0.9 upper=0.9 effort=150 velocity=1.6 -> lower=-0.9 upper=0.9 effort=100 velocity=1.5
- joint axis_y: limit lower=-0.9 upper=0.9 effort=150 velocity=1.6 -> lower=-0.9 upper=0.9 effort=100 velocity=1.5

Commit message: Reduce gripper range. This may fix the 0.07 limit error in gazebo.

File: suturo_manipulation_moveit/config/arm.urdf (robot description, URDF)
Before this commit: robot kuka_lwr, 16 links, 15 joints
Joints:
- joint joint_before_finger1: limit lower=-0.035 upper=0 effort=150 velocity=1.6 -> lower=-0.034 upper=0 effort=150 velocity=1.6
- joint joint_before_finger2: limit lower=0 upper=0.035 effort=150 velocity=1.6 -> lower=0 upper=0.034 effort=150 velocity=1.6

Commit message: reduced the limits of joint 6 even further

File: suturo_manipulation_moveit/config/arm.urdf (robot description, URDF)
Before this commit: robot kuka_lwr, 16 links, 15 joints
Joints:
- joint lwr_joint_6: limit lower=-1.7 upper=1.7 effort=150 velocity=1.6 -> lower=-1.65 upper=1.65 effort=150 velocity=1.6

Commit message: stelter: increased max gripper width

File: suturo_manipulation_moveit/config/arm.urdf (robot description, URDF)
Before this commit: robot kuka_lwr, 16 links, 15 joints
Joints:
- joint joint_before_finger1: limit lower=-0.034 upper=0 effort=150 velocity=1.6 -> lower=-0.03451 upper=0 effort=150 velocity=1.6
- joint joint_before_finger2: limit lower=0 upper=0.034 effort=150 velocity=1.6 -> lower=0 upper=0.03451 effort=150 velocity=1.6
